File: LM5116 Kicad File/LM5116.kicad_pcb (KiCad board)
At the start: 4 copper layers, 58.5 x 83.3 mm, 88 parts, among them J1 XT60-M, J10 PH1-01-UA, J11 PH1-01-UA, J12 PH1-01-UA, J13 PH1-01-UA, J14 61300311121, J15 61300311121, J16 61300311121, J17 61300311121, J18 61300311121, J19 61300311121, J2 PH1-01-UA, J20 61300311121, J21 61300311121, J22 61300311121, J23 61300311121, J24 61300311121, J25 61300311121, J3 PH1-01-UA, J4 PH1-01-UA, J5 PH1-01-UA, J6 PH1-01-UA, J7 PH1-01-UA, J8 PH1-01-UA, J9 PH1-01-UA, Q1 CSD17304Q3, Q2 CSD17304Q3, Q3 CSD17304Q3, Q4 CSD17304Q3, Q5 2N7002, Q6 IQDH29NE2LM5CG, U1 LM25116MHX/NOPB, U2 TLV1701AIDBVR, U3 TL431DBZ

Commit message: Update
Routing:
- net GNDPWR: track 80.4 -> 72.4 mm, vias 72 -> 77
- added copper zone on F.Cu, net GNDPWR
