File: LM5116 Kicad File/LM5116.kicad_pcb (KiCad board)
At the start: 4 copper layers, 58.5 x 83.3 mm, 88 parts, among them J1 XT60-M, J10 PH1-01-UA, J11 PH1-01-UA, J12 PH1-01-UA, J13 PH1-01-UA, J14 61300311121, J15 61300311121, J16 61300311121, J17 61300311121, J18 61300311121, J19 61300311121, J2 PH1-01-UA, J20 61300311121, J21 61300311121, J22 61300311121, J23 61300311121, J24 61300311121, J25 61300311121, J3 PH1-01-UA, J4 PH1-01-UA, J5 PH1-01-UA, J6 PH1-01-UA, J7 PH1-01-UA, J8 PH1-01-UA, J9 PH1-01-UA, Q1 CSD17304Q3, Q2 CSD17304Q3, Q3 CSD17304Q3, Q4 CSD17304Q3, Q5 2N7002, Q6 IQDH29NE2LM5CG, U1 LM25116MHX/NOPB, U2 TLV1701AIDBVR, U3 TL431DBZ

Commit message: Update Kicad File
Parts:
- moved C20 9.79 mm to (136.4, 93.3)
- moved C3 9.79 mm to (136.4, 88.5)
- moved C4 9.79 mm to (163.8, 77.7)
- moved D3 9.79 mm to (149.8, 82.1)
- moved D4 9.79 mm to (171.5, 121.7)
- moved J14 9.79 mm to (173.2, 129.4)
- moved J17 9.79 mm to (159.9, 129.4)
- moved J18 9.79 mm to (155.4, 129.4)
- moved J21 9.79 mm to (142.1, 129.4)
- moved J22 9.79 mm to (137.7, 129.4)
- moved J23 9.79 mm to (133.2, 129.4)
- moved Q1 9.79 mm to (151.3, 78.3)
- moved Q2 9.79 mm to (146.3, 78.3)
- moved R11 9.79 mm to (149.5, 82.1)
- moved R12 9.79 mm to (145.7, 82.1)
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Routing:
- net GND: track 21.9 -> 13.4 mm, vias 15 -> 36
- net /FB: track 13.4 -> 14.3 mm
- net /SW: track 11.1 -> 10.9 mm, vias 43 -> 38
- net Net-(R4-Pad2): vias 0 -> 1
- added copper zone on F.Cu, net GND
